File: Hydrophone_PSU.kicad_sch (KiCad schematic)
At the start: 27 parts, among them J1 Screw_Terminal_01x02, J2 Screw_Terminal_01x03, U1 LT8471IFE_PBF

Commit message: poprawki Tadeusz
Parts:
- added D3, D4: V10P10, Package_TO_SOT_SMD:TO-277A, symbol Device:D_Schottky_AAK
Connections:
- net +20VSQW: now also D3.3 (K); no longer C4.2, L1.2, R4.1
- net -20VSQW: now also D4.2 (A); no longer L2.1, R7.2, U1.19 (E2)
- net GND: now also C10.1; no longer C10.2
- net HV-: now also C10.2, D2.2 (A); no longer C10.1, D2.1 (K)
- net at T2.4: now also D2.1 (K); no longer D2.2 (A)
- new net: D4.3 (K), L2.1, R7.2, U1.19 (E2)
- new net: C4.2, D3.2 (A), L1.2, R4.1
- no-connect marks 0 -> 1
Other:
- moved on the sheet: C10, D2, J2
