File: Hydrophone_Transformer.kicad_sch (KiCad schematic)
At the start: 4 parts

Commit message: poprawki Tadeusz
Connections:
- net GND: no longer H1.1, H3.1
Changed lines of the file:
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@@
 	(generator_version "9.0")
 	(paper "A4")
-	(junction
-		(at 52.07 60.96)
-		(diameter 0)
-		(color 0 0 0 0)
-	)
-	(junction
-		(at 52.07 48.26)
-		(diameter 0)
-		(color 0 0 0 0)
-	)
 	(wire
 		(pts
@@
 		)
 		(stroke
-			(width 0)
-			(type default)
-		)
-	)
-	(wire
-		(pts
-			(xy 43.18 60.96) (xy 52.07 60.96)
-		)
-		(stroke
-			(width 0)
-			(type default)
-		)
-	)
-	(wire
-		(pts
-			(xy 43.18 48.26) (xy 52.07 48.26)
-		)
-		(stroke
